File: eagle/solar-fan.sch (EAGLE design)
At the start: 49 parts, among them Q1 MMBT2222A, Q2 MMBT2222A, Q3 MMBT2222A, U1 LT3652, U2 ATTINY85

Commit message: minor electronics/software updates, still rev A
Parts:
- +5V: PN2 811-2196-5-ND -> LM7805CT-ND
- BAT, SUN: PN (none) -> 277-1667-ND
- R1: value 430k -> 560K; PN P430KGCT-ND -> P560KGCT-ND
Changed lines of the file:
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@@
 <attribute name="PN" value="MBRS140T3GOSCT-ND"/>
 </part>
-<part name="R1" library="SparkFun-Passives" deviceset="RESISTOR" device="0603-RES" value="430k">
-<attribute name="PN" value="P430KGCT-ND"/>
+<part name="R1" library="SparkFun-Passives" deviceset="RESISTOR" device="0603-RES" value="560K">
+<attribute name="PN" value="P560KGCT-ND"/>
 </part>
 <part name="R2" library="SparkFun-Passives" deviceset="RESISTOR" device="0603-RES" value="100k">
@@
 <part name="+5V" library="SparkFun-Connectors" deviceset="M03" device="PTH" value="7805">
 <attribute name="PN" value="811-2196-5-ND"/>
-<attribute name="PN2" value="811-2196-5-ND"/>
+<attribute name="PN2" value="LM7805CT-ND"/>
 </part>
 <part name="SUPPLY3" library="SparkFun-Aesthetics" deviceset="V_BATT" device=""/>
@@
 <attribute name="PN" value="SZBZX84C6V2LT1GOSCT-ND"/>
 </part>
-<part name="SUN" library="SparkFun-Connectors" deviceset="M02" device="5MM"/>
-<part name="BAT" library="SparkFun-Connectors" deviceset="M02" device="5MM"/>
+<part name="SUN" library="SparkFun-Connectors" deviceset="M02" device="5MM">
+<attribute name="PN" value="277-1667-ND"/>
+</part>
+<part name="BAT" library="SparkFun-Connectors" deviceset="M02" device="5MM">
+<attribute name="PN" value="277-1667-ND"/>
+</part>
 <part name="GND3" library="SparkFun-Aesthetics" deviceset="GND" device=""/>
 <part name="GND6" library="SparkFun-Aesthetics" deviceset="GND" device=""/>
@@
 <attribute name="PN" x="119.38" y="38.1" size="1.778" layer="96" display="off"/>
 </instance>
-<instance part="SUN" gate="G$1" x="12.7" y="40.64"/>
-<instance part="BAT" gate="G$1" x="0" y="58.42"/>
+<instance part="SUN" gate="G$1" x="12.7" y="40.64">
+<attribute name="PN" x="12.7" y="40.64" size="1.778" layer="96" display="off"/>
+</instance>
+<instance part="BAT" gate="G$1" x="0" y="58.42">
+<attribute name="PN" x="0" y="58.42" size="1.778" layer="96" display="off"/>
+</instance>
 <instance part="GND3" gate="1" x="20.32" y="53.34"/>
 <instance part="GND6" gate="1" x="22.86" y="35.56"/>
